File: schematic/Prototype1.kicad_pcb (KiCad board)
At the start: 2 copper layers, 95 x 72 mm, 19 parts, among them J1 Conn_AVR_UPDI, J3 Conn_I2C_Master, SW1 TSD1265, U1 ATmega4809-P, U2 HM628128DLP-5, U3 Z84C00

Commit message: Migrate to KiCad 6.0
Connections:
- net /~BUSACK~ renamed /~{BUSACK}
- net /~BUSREQ~ renamed /~{BUSREQ}
- net /~DBG_RESET~ renamed /~{DBG_RESET}
- net /~DBG_RTS~ renamed /~{DBG_RTS}
- net /~INT~ renamed /~{INT}
- net /~IORQ~ renamed /~{IORQ}
- net /~M1~ renamed /~{M1}
- net /~MREQ~ renamed /~{MREQ}
- net /~NMI~ renamed /~{NMI}
- net /~RAM_E~ renamed /~{RAM_E}
- net /~RD~ renamed /~{RD}
- net /~RESET~ renamed /~{RESET}
- net /~USR_LED~ renamed /~{USR_LED}
- net /~USR_SW~ renamed /~{USR_SW}
- net /~WAIT~ renamed /~{WAIT}
- net /~WR~ renamed /~{WR}
Other:
- net class Default removed
