File: schematic/Prototype1.kicad_sch (KiCad schematic)
At the start: 15 parts, among them J1 Conn_AVR_UPDI, J3 Conn_I2C_Master, SW1 TSD1265, U1 ATmega4809-P, U2 HM628128DLP-5, U3 Z84C00

Commit message: Satisfy Electrical Rules Checker
Parts:
- added B1: Micro_SD, 0-LocalLibrary:uSD_CARD, symbol 0-LocalLibrary:Micro_SD
Connections:
- net GND: now also B1.7 (GND)
- net SD_DI: now also B1.3 (DI)
- net SD_DO: now also B1.5 (DO)
- net SD_SCK: now also B1.4 (SCK)
- net VCC: now also B1.1 (VCC)
- net ~{SD_CS}: now also B1.2 (~{CS})
Changed lines of the file:
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@@
     (effects (font (size 1.27 1.27)) (justify right bottom))
+  )
+  (label "D[0..7]" (at 107.95 29.21 0)
+    (effects (font (size 1.27 1.27)) (justify left bottom))
   )
   (label "CLK" (at 80.01 88.9 0)
@@
   (label "A10" (at 152.4 77.47 180)
     (effects (font (size 1.27 1.27)) (justify right bottom))
+  )
+  (label "A[0..15]" (at 107.95 31.75 0)
+    (effects (font (size 1.27 1.27)) (justify left bottom))
   )
   (label "~{IORQ}" (at 46.99 53.34 180)
@@
     )
     (property "Datasheet" "" (id 3) (at 128.27 99.06 0)
-      (effects (font (size 1.27 1.27)) hide)
-    )
-    (pin "1")
-  )
-  (symbol (lib_id "power:VCC") (at -1352.55 -1136.65 0) (unit 1)
-    (in_bom yes) (on_board yes)
-    (property "Reference" "#PWR01" (id 0) (at -1352.55 -1132.84 0)
-      (effects (font (size 1.27 1.27)) hide)
-    )
-    (property "Value" "VCC" (id 1) (at -1352.1182 -1141.0442 0))
-    (property "Footprint" "" (id 2) (at -1352.55 -1136.65 0)
-      (effects (font (size 1.27 1.27)) hide)
-    )
-    (property "Datasheet" "" (id 3) (at -1352.55 -1136.65 0)
       (effects (font (size 1.27 1.27)) hide)
     )
@@
     (pin "1")
   )
+  (symbol (lib_id "0-LocalLibrary:Micro_SD") (at 62.23 152.4 0) (unit 1)
+    (in_bom yes) (on_board yes)
+    (property "Reference" "B1" (id 0) (at 60.96 142.24 0)
+      (effects (font (size 1.27 1.27)) (justify left))
+    )
+    (property "Value" "Micro_SD" (id 1) (at 62.23 163.83 0)
+      (effects (font (size 1.27 1.27)) (justify left))
+    )
+    (property "Footprint" "0-LocalLibrary:uSD_CARD" (id 2) (at 62.23 152.4 0)
+      (effects (font (size 1.27 1.27)) hide)
+    )
+    (property "Datasheet" "~" (id 3) (at 62.23 152.4 0)
+      (effects (font (size 1.27 1.27)) hide)
+    )
+    (pin "1")
+    (pin "2")
+    (pin "3")
+    (pin "4")
+    (pin "5")
+    (pin "6")
+    (pin "7")
+  )
   (sheet_instances
     (path "/" (page "1"))
   )
   (symbol_instances
-    (path "/00000000-0000-0000-0000-00005cde46a4"
-      (reference "#PWR01") (unit 1) (value "VCC") (footprint "")
-    )
     (path "/00000000-0000-0000-0000-00005ce5efde"
       (reference "#PWR02") (unit 1) (value "VCC") (footprint "")
@@
       (reference "#PWR0101") (unit 1) (value "VCC") (footprint "")
     )
+    (path "/9947d1f2-3080-4104-ba9f-a97b668bb725"
+      (reference "B1") (unit 1) (value "Micro_SD") (footprint "0-LocalLibrary:uSD_CARD")
+    )
     (path "/00000000-0000-0000-0000-00005ea154e8"
